Commit message: works for 2 bittles

File: source/BittleHRL/BittleHRL/tasks/direct/bittlehrl/Bittle_URDF/urdf/bittle.urdf (robot description, URDF)
Before this commit: robot bittle, 13 links, 12 joints
Joints:
- joint left-back-knee-joint: limit lower=-2.182 upper=2.182 effort=1.0 velocity=1.5708 -> lower=-1.22173 upper=1.48353 effort=1.0 velocity=1.5708
- joint left-back-shoulder-joint: limit lower=-2.182 upper=2.182 effort=1.0 velocity=1.5708 -> lower=-1.5708 upper=1.22173 effort=1.0 velocity=1.5708
- joint left-front-knee-joint: limit lower=-2.182 upper=2.182 effort=1.0 velocity=1.5708 -> lower=-1.22173 upper=1.48353 effort=1.0 velocity=1.5708
- joint left-front-shoulder-joint: limit lower=-2.182 upper=2.182 effort=1.0 velocity=1.5708 -> lower=-1.5708 upper=1.22173 effort=1.0 velocity=1.5708
- joint right-back-knee-joint: limit lower=-2.182 upper=2.182 effort=1.0 velocity=1.5708 -> lower=-1.22173 upper=1.48353 effort=1.0 velocity=1.5708
- joint right-front-knee-joint: limit lower=-2.182 upper=2.182 effort=1.0 velocity=1.5708 -> lower=-1.22173 upper=1.48353 effort=1.0 velocity=1.5708
- joint right-front-shoulder-joint: limit lower=-2.182 upper=2.182 effort=1.0 velocity=1.5708 -> lower=-1.5708 upper=1.22173 effort=1.0 velocity=1.5708

Commit message: fixed the joint angle bugs

File: source/BittleHRL/BittleHRL/tasks/direct/bittlehrl/Bittle_URDF/urdf/bittle.urdf (robot description, URDF)
Before this commit: robot bittle, 13 links, 12 joints
Joints:
- joint left-back-knee-joint: limit lower=-1.22173 upper=1.48353 effort=1.0 velocity=1.5708 -> lower=-2.182 upper=2.182 effort=1.0 velocity=1.5708
- joint left-back-shoulder-joint: limit lower=-1.5708 upper=1.22173 effort=1.0 velocity=1.5708 -> lower=-2.182 upper=2.182 effort=1.0 velocity=1.5708
- joint left-front-knee-joint: limit lower=-1.22173 upper=1.48353 effort=1.0 velocity=1.5708 -> lower=-2.182 upper=2.182 effort=1.0 velocity=1.5708
- joint left-front-shoulder-joint: limit lower=-1.5708 upper=1.22173 effort=1.0 velocity=1.5708 -> lower=-2.182 upper=2.182 effort=1.0 velocity=1.5708
- joint right-back-knee-joint: limit lower=-1.22173 upper=1.48353 effort=1.0 velocity=1.5708 -> lower=-2.182 upper=2.182 effort=1.0 velocity=1.5708
- joint right-back-shoulder-joint: limit lower=-1.5708 upper=1.22173 effort=1.0 velocity=1.5708 -> lower=-2.182 upper=2.182 effort=1.0 velocity=1.5708
- joint right-front-knee-joint: limit lower=-1.22173 upper=1.48353 effort=1.0 velocity=1.5708 -> lower=-2.182 upper=2.182 effort=1.0 velocity=1.5708
- joint right-front-shoulder-joint: limit lower=-1.5708 upper=1.22173 effort=1.0 velocity=1.5708 -> lower=-2.182 upper=2.182 effort=1.0 velocity=1.5708

Commit message: added terrain randomization with random frictions, fixed URDF

File: source/BittleHRL/BittleHRL/tasks/direct/bittlehrl/Bittle_URDF/urdf/bittle.urdf (robot description, URDF)
Before this commit: robot bittle, 13 links, 12 joints
Joints:
- joint left-back-knee-joint: limit lower=-2.182 upper=2.182 effort=1.0 velocity=1.5708 -> lower=-1.22173 upper=1.48353 effort=1.0 velocity=1.5708
- joint left-back-shoulder-joint: limit lower=-2.182 upper=2.182 effort=1.0 velocity=1.5708 -> lower=-1.5708 upper=1.22173 effort=1.0 velocity=1.5708
- joint left-front-knee-joint: limit lower=-2.182 upper=2.182 effort=1.0 velocity=1.5708 -> lower=-1.22173 upper=1.48353 effort=1.0 velocity=1.5708
- joint left-front-shoulder-joint: limit lower=-2.182 upper=2.182 effort=1.0 velocity=1.5708 -> lower=-1.5708 upper=1.22173 effort=1.0 velocity=1.5708
- joint right-back-knee-joint: limit lower=-2.182 upper=2.182 effort=1.0 velocity=1.5708 -> lower=-1.22173 upper=1.48353 effort=1.0 velocity=1.5708
- joint right-back-shoulder-joint: limit lower=-2.182 upper=2.182 effort=1.0 velocity=1.5708 -> lower=-1.5708 upper=1.22173 effort=1.0 velocity=1.5708
- joint right-front-knee-joint: limit lower=-2.182 upper=2.182 effort=1.0 velocity=1.5708 -> lower=-1.22173 upper=1.48353 effort=1.0 velocity=1.5708
- joint right-front-shoulder-joint: limit lower=-2.182 upper=2.182 effort=1.0 velocity=1.5708 -> lower=-1.5708 upper=1.22173 effort=1.0 velocity=1.5708
